File: egj-gamepacks-2025/RP2350.kicad_sch (KiCad schematic)
At the start: 40 parts, among them J2 Conn_01x03_Pin, SW1 SW_Push, SW2 SW_Push, U1 W25Q128JVS, U2 DNF, U4 RP2350_80QFN, Y1 ABM8-272-T3

Commit message: UPDATE: sync local schematic and board work
Parts:
- removed J2: Conn_01x03_Pin, Connector_PinHeader_2.54mm:PinHeader_1x03_P2.54mm_Horizontal, symbol Connector:Conn_01x03_Pin
- added J3: SM03B-SRSS-TB, Connector_JST:JST_SH_SM03B-SRSS-TB_1x03-1MP_P1.00mm_Horizontal, symbol Connector_Generic_MountingPin:Conn_01x03_MountingPin
- added U5: USBLC6-2P6, Package_TO_SOT_SMD:SOT-666, symbol Power_Protection:USBLC6-2P6
Connections:
- net GBA_ADD0: now also U4.6 (GPIO8); no longer U4.1 (GPIO4)
- net GBA_ADD1: now also U4.7 (GPIO9); no longer U4.2 (GPIO5)
- net GBA_ADD10: now also U4.18 (GPIO18); no longer U4.13 (GPIO14)
- net GBA_ADD11: now also U4.19 (GPIO19); no longer U4.14 (GPIO15)
- net GBA_ADD12: now also U4.20 (GPIO20); no longer U4.16 (GPIO16)
- net GBA_ADD13: now also U4.21 (GPIO21); no longer U4.17 (GPIO17)
- net GBA_ADD14: now also U4.22 (GPIO22); no longer U4.18 (GPIO18)
- net GBA_ADD15: now also U4.23 (GPIO23); no longer U4.19 (GPIO19)
- net GBA_ADD2: now also U4.8 (GPIO10); no longer U4.3 (GPIO6)
- net GBA_ADD3: now also U4.9 (GPIO11); no longer U4.4 (GPIO7)
- net GBA_ADD4: now also U4.11 (GPIO12); no longer U4.6 (GPIO8)
- net GBA_ADD5: now also U4.12 (GPIO13); no longer U4.7 (GPIO9)
- net GBA_ADD6: now also U4.13 (GPIO14); no longer U4.8 (GPIO10)
- net GBA_ADD7: now also U4.14 (GPIO15); no longer U4.9 (GPIO11)
- net GBA_ADD8: now also U4.16 (GPIO16); no longer U4.11 (GPIO12)
- net GBA_ADD9: now also U4.17 (GPIO17); no longer U4.12 (GPIO13)
- net GBA_DATA0: now also U4.77 (GPIO0); no longer U4.20 (GPIO20)
- net GBA_DATA1: now also U4.78 (GPIO1); no longer U4.21 (GPIO21)
- net GBA_DATA2: now also U4.79 (GPIO2); no longer U4.22 (GPIO22)
- net GBA_DATA3: now also U4.80 (GPIO3); no longer U4.23 (GPIO23)
- net GBA_DATA4: now also U4.1 (GPIO4); no longer U4.25 (GPIO24)
- net GBA_DATA5: now also U4.2 (GPIO5); no longer U4.26 (GPIO25)
- net GBA_DATA6: now also U4.3 (GPIO6); no longer U4.27 (GPIO26)
- net GBA_DATA7: now also U4.4 (GPIO7); no longer U4.28 (GPIO27)
- net GBA_SIG.N_CS: now also U4.28 (GPIO27); no longer U4.80 (GPIO3)
- net GBA_SIG.N_RD: now also U4.27 (GPIO26); no longer U4.79 (GPIO2)
- net GBA_SIG.N_WR: now also U4.26 (GPIO25); no longer U4.78 (GPIO1)
- net GBA_SIG.PHI: now also U4.25 (GPIO24); no longer U4.77 (GPIO0)
- net GND: now also J3.2 (Pin_2), J3.MP (MountPin), U5.2 (GND)
- net SWCLK: now also J3.1 (Pin_1)
- net SWD: now also J3.3 (Pin_3)
- net USB.USB_D_C+: now also U5.1 (I/O1); no longer R10.1
- net USB.USB_D_C-: now also U5.3 (I/O2); no longer R11.1
- net +3V3_USB: no longer names the net of U4.58 (GPIO47_ADC7)
- new net USB_D+: R10.1, U5.6 (I/O1)
- new net USB_D-: R11.1, U5.4 (I/O2)
- new net VBUS: U5.5 (VBUS)
- no-connect marks 7 -> 8
Other:
- note added: "JST Debug Connector"

Commit message: FIX: schematic fixes, JLCPCB parts with LCSC numbers and GBA bus GPIO remap
Parts:
- added R23, R24: 100k, Resistor_SMD:R_0402_1005Metric, symbol Device:R
- C10, C11, C7, C8: LCSC (none) -> C23733
- C12, C13, C14, C15, C16, C17, C18, C19, C2, C21, C22, C9: LCSC (none) -> C1525
- C20: LCSC (none) -> C15850
- C4, C5: LCSC (none) -> C1548
- J3: value SM03B-SRSS-TB -> BM03B-SRSS-TB; footprint Connector_JST:JST_SH_SM03B-SRSS-TB_1x03-1MP_P1.00mm_Horizontal -> Connector_JST:JST_SH_BM03B-SRSS-TB_1x03-1MP_P1.00mm_Vertical; LCSC (none) -> C160389
- L1: LCSC (none) -> C98336
- R10, R11: LCSC (none) -> C25100
- R12: LCSC (none) -> C25744
- R2: LCSC (none) -> C17168
- R6, R7, R9: LCSC (none) -> C11702
- R8: LCSC (none) -> C25105
- SW1, SW2: value SW_Push -> PTS810SJG250SMTRLFS; footprint Button_Switch_SMD:SW_Push_1P1T_NO_Vertical_Wuerth_434133025816 -> Button_Switch_SMD:SW_SPST_PTS810; LCSC (none) -> C221895
- U1: value W25Q128JVS -> W25Q128JVSIQ; LCSC (none) -> C97521
- U4: LCSC (none) -> C42415655
- U5: LCSC (none) -> C15999
- Y1: LCSC (none) -> C20625731
Connections:
- net +3V3_GBA: now also R23.1; no longer U4.57 (GPIO46_ADC6)
- net GBA_ADD0: now also U4.1 (GPIO4); no longer U4.6 (GPIO8)
- net GBA_ADD1: now also U4.2 (GPIO5); no longer U4.7 (GPIO9)
- net GBA_ADD10: now also U4.13 (GPIO14); no longer U4.18 (GPIO18)
- net GBA_ADD11: now also U4.14 (GPIO15); no longer U4.19 (GPIO19)
- net GBA_ADD12: now also U4.16 (GPIO16); no longer U4.20 (GPIO20)
- net GBA_ADD13: now also U4.17 (GPIO17); no longer U4.21 (GPIO21)
- net GBA_ADD14: now also U4.18 (GPIO18); no longer U4.22 (GPIO22)
- net GBA_ADD15: now also U4.19 (GPIO19); no longer U4.23 (GPIO23)
- net GBA_ADD2: now also U4.3 (GPIO6); no longer U4.8 (GPIO10)
- net GBA_ADD3: now also U4.4 (GPIO7); no longer U4.9 (GPIO11)
- net GBA_ADD4: now also U4.6 (GPIO8); no longer U4.11 (GPIO12)
- net GBA_ADD5: now also U4.7 (GPIO9); no longer U4.12 (GPIO13)
- net GBA_ADD6: now also U4.8 (GPIO10); no longer U4.13 (GPIO14)
- net GBA_ADD7: now also U4.9 (GPIO11); no longer U4.14 (GPIO15)
- net GBA_ADD8: now also U4.11 (GPIO12); no longer U4.16 (GPIO16)
- net GBA_ADD9: now also U4.12 (GPIO13); no longer U4.17 (GPIO17)
- net GBA_DATA0: now also U4.20 (GPIO20); no longer U4.77 (GPIO0)
- net GBA_DATA1: now also U4.21 (GPIO21); no longer U4.78 (GPIO1)
- net GBA_DATA2: now also U4.22 (GPIO22); no longer U4.79 (GPIO2)
- net GBA_DATA3: now also U4.23 (GPIO23); no longer U4.80 (GPIO3)
- net GBA_DATA4: now also U4.25 (GPIO24); no longer U4.1 (GPIO4)
- net GBA_DATA5: now also U4.26 (GPIO25); no longer U4.2 (GPIO5)
- net GBA_DATA6: now also U4.27 (GPIO26); no longer U4.3 (GPIO6)
- net GBA_DATA7: now also U4.28 (GPIO27); no longer U4.4 (GPIO7)
- net GBA_SIG.N_CS: now also U4.80 (GPIO3); no longer U4.28 (GPIO27)
- net GBA_SIG.N_RD: now also U4.79 (GPIO2); no longer U4.27 (GPIO26)
- net GBA_SIG.N_WR: now also U4.78 (GPIO1); no longer U4.26 (GPIO25)
- net GBA_SIG.PHI: now also U4.77 (GPIO0); no longer U4.25 (GPIO24)
- net GND: now also R24.2
- new net: R23.2, R24.1, U4.57 (GPIO46_ADC6)

Commit message: FIX: RP2350 regulator inductor, I2C pull-ups, DVDD decoupling and drop second flash option
Parts:
- removed C3: DNF, Capacitor_SMD:C_0402_1005Metric, symbol Device:C
- removed R1, R3, R5: DNF, Resistor_SMD:R_0402_1005Metric, symbol Device:R
- removed U2: DNF, Package_SO:SOIC-8_5.3x5.3mm_P1.27mm, symbol Memory_Flash:W25Q128JVS
- added C33: 100n, Capacitor_SMD:C_0402_1005Metric, symbol Device:C
- L1: value 3.3u -> AOTA-B201610S3R3-101-T; LCSC C98336 -> C42411119
- R4: now not fitted; now left out of the parts list
Connections:
- net +1V1: now also C33.1
- net GND: now also C33.2
