File: egj-gamepacks-2025/untitled.kicad_sch (KiCad schematic)
At the start: 24 parts, among them U11 VL6180XV0NR_1, U12 TXS0108EPW, U14 BNO055

Commit message: UPDATE: sync local schematic and board work
Connections:
- net +1V8 renamed +2V8
Changed lines of the file:
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@@
 	)
 	(symbol
-		(lib_id "power:+1V8")
+		(lib_id "power:+2V8")
 		(at 161.29 41.91 0)
 		(unit 1)
@@
 			)
 		)
-		(property "Value" "+1V8"
+		(property "Value" "+2V8"
 			(at 161.29 36.83 0)
 			(effects
@@
 			)
 		)
-		(property "Description" "Power symbol creates a global label with name \"+1V8\""
+		(property "Description" "Power symbol creates a global label with name \"+2V8\""
 			(at 161.29 41.91 0)
 			(effects
@@
 	)
 	(symbol
-		(lib_id "power:+1V8")
+		(lib_id "power:+2V8")
 		(at 35.56 130.81 0)
 		(unit 1)
@@
 			)
 		)
-		(property "Value" "+1V8"
+		(property "Value" "+2V8"
 			(at 35.56 125.73 0)
 			(effects
@@
 			)
 		)
-		(property "Description" "Power symbol creates a global label with name \"+1V8\""
+		(property "Description" "Power symbol creates a global label with name \"+2V8\""
 			(at 35.56 130.81 0)
 			(effects
@@
 	)
 	(symbol
-		(lib_id "power:+1V8")
+		(lib_id "power:+2V8")
 		(at 132.08 148.59 0)
 		(unit 1)
@@
 			)
 		)
-		(property "Value" "+1V8"
+		(property "Value" "+2V8"
 			(at 132.08 143.51 0)
 			(effects
@@
 			)
 		)
-		(property "Description" "Power symbol creates a global label with name \"+1V8\""
+		(property "Description" "Power symbol creates a global label with name \"+2V8\""
 			(at 132.08 148.59 0)
 			(effects

Commit message: FIX: schematic fixes, JLCPCB parts with LCSC numbers and GBA bus GPIO remap
Parts:
- C26, C27, C30: LCSC (none) -> C28323
- C28, C32: LCSC (none) -> C49678
- C29: LCSC (none) -> C1779
- C31: LCSC (none) -> C113854
- R13, R14, R17, R18, R19, R21: LCSC (none) -> C25900
- R15, R16: LCSC (none) -> C25105
- R20, R22: LCSC (none) -> C25744
- TP3, TP4, TP5, TP6: LCSC (none) -> C2906768
- U11: value VL6180XV0NR_1 -> VL6180V1NR/1; LCSC (none) -> C2655167
- U12: LCSC (none) -> C17206
- U14: LCSC (none) -> C93216
Connections:
- net +3V3: now also R22.1; no longer R22.2, U14.11 (~{RESET})
- net BNO055_UART.RESET: now also R22.2, U14.11 (~{RESET}); no longer R22.1

Commit message: FIX: RP2350 regulator inductor, I2C pull-ups, DVDD decoupling and drop second flash option
Parts:
- R13, R14: value 4.7K -> 10K; LCSC C25900 -> C25744
- R17, R18: value 4.7K -> 47K; LCSC C25900 -> C25792
Changed lines of the file:
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@@
 			)
 		)
-		(property "Value" "4.7K"
+		(property "Value" "47K"
 			(at 55.88 138.4299 0)
 			(effects
@@
 			)
 		)
-		(property "LCSC" "C25900"
+		(property "LCSC" "C25792"
 			(at 53.34 137.16 0)
 			(effects
@@
 			)
 		)
-		(property "Value" "4.7K"
+		(property "Value" "47K"
 			(at 43.18 138.4299 0)
 			(effects
@@
 			)
 		)
-		(property "LCSC" "C25900"
+		(property "LCSC" "C25792"
 			(at 45.72 137.16 0)
 			(effects
@@
 			)
 		)
-		(property "Value" "4.7K"
+		(property "Value" "10K"
 			(at 71.12 138.4299 0)
 			(effects
@@
 			)
 		)
-		(property "LCSC" "C25900"
+		(property "LCSC" "C25744"
 			(at 73.66 137.16 0)
 			(effects
@@
 			)
 		)
-		(property "Value" "4.7K"
+		(property "Value" "10K"
 			(at 83.82 138.4299 0)
 			(effects
@@
 			)
 		)
-		(property "LCSC" "C25900"
+		(property "LCSC" "C25744"
 			(at 81.28 137.16 0)
 			(effects
